File: temp-humidity sensor.kicad_pcb (KiCad board)
At the start: 2 copper layers, 36 parts, among them J1 Conn_01x02, J2 USB_C_Receptacle_USB2.0_16P, SW1 SW_Push, SW2 SW_Push, SW3 SS-12D01-G040, U1 SHT4x, U2 ESP32-C6-WROOM-1, U3 BQ24074RGT, U4 USBLC6-2SC6, U5 TPS63031DSK

Commit message: Working On PCB
Parts:
- added C11: 470n, Capacitor_SMD:C_0603_1608Metric, F.Cu at (105.4, 94.6)
- added C12: 470n, Capacitor_SMD:C_0603_1608Metric, F.Cu at (108.6, 94.6)
- added R15: 0R, Resistor_SMD:R_0603_1608Metric, F.Cu at (107.0, 94.6)
- C10: value 10u -> 100n
- moved R9 56.0 mm to (106.2, 102.1), turned to 180 degrees
- moved R10 52.5 mm to (102.8, 88.6)
- moved R12 51.2 mm to (102.5, 86.1), turned to -90 degrees
- moved U3 49.1 mm to (106.8, 87.4), turned to 180 degrees
- moved U5 48.4 mm to (112.5, 80.4)
- moved R11 47.2 mm to (108.3, 91.1), turned to 90 degrees
- moved J2 46.6 mm to (98.6, 99.6), turned to -90 degrees
- moved R7 45.7 mm to (106.1, 97.1), turned to 180 degrees
- moved R13 42.8 mm to (113.8, 98.4), turned to 180 degrees
- moved R14 42.7 mm to (113.8, 100.6), turned to 180 degrees
- moved R8 39.4 mm to (110.2, 89.8), turned to -90 degrees
- moved C7 37.6 mm to (109.3, 82.7)
- moved L1 37.4 mm to (106.3, 76.6), turned to 90 degrees
- moved J1 36.8 mm to (114.2, 90.0), turned to 90 degrees
- moved C5 36.5 mm to (105.8, 90.6)
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Connections:
- C5 pad 1: /VBUS -> /VBUSF
- J1 pad 1: /BAT- -> Earth
- U2 pad 15: unconnected-(U2-GPIO9-Pad15) -> /GPIO9
- U3 pad 13: /VBUS -> /VBUSF
Routing:
- net +3V3: track 0.00 -> 11.5 mm
- net Net-(U5-L2): track 0.00 -> 9.57 mm
- net +5V: track 0.00 -> 7.45 mm
- net /VOUT: track 0.00 -> 6.65 mm
- net /VBUS: track 0.00 -> 5.79 mm
- net /VBUSF: track 0.00 -> 5.57 mm
- net Net-(U5-L1): track 0.00 -> 5.51 mm
- net /BAT+: track 0.00 -> 4.02 mm
- net /CHIP_PU: track 0.00 -> 2.89 mm
- net Net-(U5-EN): track 0.00 -> 2.52 mm
- net Earth: vias 0 -> 11
- added copper zone on B.Cu, net Earth
Other:
- board outline added: 70.4 x 34.8 mm

Commit message: Finished Design
Parts:
- removed R13, R14: 22R, Resistor_SMD:R_0603_1608Metric
- added TP2: TestPoint, TestPoint:TestPoint_Pad_D1.0mm, F.Cu at (162.4, 94.9)
- added TP3: TestPoint, TestPoint:TestPoint_Pad_D1.0mm, F.Cu at (98.3, 82.0)
- added TP4: TestPoint, TestPoint:TestPoint_Pad_D1.0mm, F.Cu at (116.2, 74.7)
- added TP5: TestPoint, TestPoint:TestPoint_Pad_D1.0mm, F.Cu at (120.7, 87.5)
- added TP6: TestPoint, TestPoint:TestPoint_Pad_D1.0mm, F.Cu at (124.2, 75.4)
- SW3: footprint LCSC:SW-TH_SS-12D01-GX -> easyeda2kicad:SW-TH_SS-12D01-GX
- moved U4 1.87 mm to (108.1, 99.6)
- moved R7 0.38 mm to (106.4, 96.8)
Connections:
- net +5V renamed VSYS
- U4 pad 4: Net-(R14-Pad2) -> /USBD+
- U4 pad 6: Net-(R13-Pad2) -> /USBD-
Routing:
- net +3V3: track 11.5 -> 101.5 mm
- net Earth: track 0.00 -> 52.9 mm, vias 11 -> 87
- net /SCL: track 0.00 -> 33.3 mm
- net /SDA: track 0.00 -> 33.0 mm
- net /USBD-: track 0.00 -> 31.9 mm
- net /USBD+: track 0.00 -> 31.9 mm
- net VSYS: track 7.45 -> 28.3 mm
- net /GPIO9: track 0.00 -> 14.0 mm
- net /VBUS: track 5.79 -> 19.0 mm
- net /BAT+: track 4.02 -> 16.2 mm
- net /CHIP_PU: track 2.89 -> 14.7 mm, vias 0 -> 2
- net /VOUT: track 6.65 -> 18.4 mm
- net /USBCD-: track 0.00 -> 8.63 mm
- net /USBCD+: track 0.00 -> 7.31 mm
- net Net-(D1-A): track 0.00 -> 4.26 mm
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- added copper zone on F.Cu, net Earth
Other:
- board text added: "+"
- board text added: "-"
- board text added: "3V3"
- board text added: "BAT"
- board text added: "OFF"
- board text added: "ON"
- board text added: "RESET"
- board text added: "VOUT"
- board text added: "VSYS"

Commit message: V3
Parts:
- removed SW3: SS-12D01-G040, easyeda2kicad:SW-TH_SS-12D01-GX
- removed TP6: TestPoint, TestPoint:TestPoint_Pad_D1.0mm
- added U6: SS12D10G5, easyeda2kicad:SW-TH_SHOU-HAN_SS12D10G4, F.Cu at (86.5, 51.2)
- C1, C2, C5, C7, C9: footprint Capacitor_SMD:C_0603_1608Metric -> Capacitor_SMD:C_0805_2012Metric
- C10: value 100n -> 10u; footprint Capacitor_SMD:C_0603_1608Metric -> Capacitor_SMD:C_0805_2012Metric
- C6: value 10u -> 4.7u; footprint Capacitor_SMD:C_0603_1608Metric -> Capacitor_SMD:C_0805_2012Metric
- R10: value 1.2K -> 1.3K
- R11: value 680R -> 698R
- U2: footprint PCM_Espressif_1:ESP32-C6-WROOM-1 -> PCM_Espressif:ESP32-C6-WROOM-1
- moved U1 113.2 mm to (257.9, 160.1)
- moved TP2 111.1 mm to (269.5, 124.5)
- moved R5 108.9 mm to (261.9, 131.8), turned to 0 degrees
- moved R4 107.8 mm to (261.9, 129.2), turned to 0 degrees
- moved R2 106.7 mm to (261.9, 124.2), turned to 0 degrees
- moved R3 103.6 mm to (261.9, 126.7)
- moved C4 100.7 mm to (257.9, 126.7), turned to 0 degrees
- moved J1 67.1 mm to (69.2, 40.2), turned to -90 degrees
- moved TP5 65.0 mm to (73.5, 42.8), turned to 180 degrees
- moved R8 57.9 mm to (77.8, 41.8), turned to 90 degrees
- moved R11 56.9 mm to (79.5, 42.0), turned to -90 degrees
- moved C6 56.7 mm to (75.8, 41.8)
- moved U3 51.2 mm to (76.4, 46.1), turned to -90 degrees
- moved C5 51.0 mm to (81.0, 46.0), turned to 90 degrees
- moved R10 45.1 mm to (80.3, 49.5), turned to 180 degrees
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Connections:
- net /CHIP_PU renamed CHIP_PU
- net /GPIO9 renamed GPIO9
- net /SCL renamed SCL
- net /SDA renamed SDA
- net /USBD+ renamed USBD+
- net /USBD- renamed USBD-
- C10 pad 1: /VOUT -> +3V3
- C7 pad 1: VSYS -> /VIN
- C9 pad 1: /VOUT -> +3V3
- R12 pad 2: VSYS -> VCC
- TP3 pad 1: VSYS -> VCC
- TP4 pad 1: /VOUT -> +3V3
- U3 pad 10: VSYS -> VCC
- U3 pad 11: VSYS -> VCC
- U3 pad 5: VSYS -> VCC
- U5 pad 1: /VOUT -> +3V3
- U5 pad 10: /VOUT -> +3V3
- U5 pad 5: VSYS -> /VIN
Routing:
- net +3V3: track 101.5 -> 0.00 mm, vias 0 -> 2
- net Earth: track 52.9 -> 0.00 mm, vias 87 -> 20
- net SCL: track 33.3 -> 0.00 mm
- net SDA: track 33.0 -> 0.00 mm
- net USBD-: track 31.9 -> 0.00 mm
- net USBD+: track 31.9 -> 0.00 mm
- net VSYS: track 28.3 -> 0.00 mm
- net /VBUS: track 19.0 -> 0.00 mm
- net /VOUT: track 18.4 -> 0.00 mm
- net /BAT+: track 16.2 -> 0.00 mm
- net CHIP_PU: track 14.7 -> 0.00 mm, vias 2 -> 0
- net GPIO9: track 14.0 -> 0.00 mm
- net Net-(U5-L2): track 9.74 -> 0.00 mm
- net /USBCD-: track 8.63 -> 0.00 mm
- net /VBUSF: track 7.80 -> 0.00 mm
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- removed copper zone on B.Cu, net Earth
- removed copper zone on F.Cu, net Earth
Other:
- board outline removed
- board text removed: "+"
- board text removed: "-"
- board text removed: "3V3"
- board text removed: "BAT"
- board text removed: "OFF"
- board text removed: "ON"
- board text removed: "RESET"
- board text removed: "VOUT"
- board text removed: "VSYS"

Commit message: Update to V3
Parts:
- added TP6: TestPoint, TestPoint:TestPoint_Pad_D1.0mm, F.Cu at (74.2, 38.2)
- added TP7: TestPoint, TestPoint:TestPoint_Pad_D1.0mm, F.Cu at (101.5, 39.0)
- added TP8: TestPoint, TestPoint:TestPoint_Pad_D1.0mm, F.Cu at (131.5, 64.5)
- added TP9: TestPoint, TestPoint:TestPoint_Pad_D1.0mm, F.Cu at (69.8, 50.2)
- moved U1 165.3 mm to (126.0, 60.6)
- moved R5 157.9 mm to (121.2, 60.0), turned to 180 degrees
- moved R4 156.1 mm to (121.2, 61.5), turned to 180 degrees
- moved TP2 152.8 mm to (130.2, 61.5)
- moved R2 152.7 mm to (123.8, 59.2), turned to 90 degrees
- moved R3 152.4 mm to (123.8, 62.4), turned to -90 degrees
- moved C4 145.5 mm to (128.2, 60.8), turned to 90 degrees
- moved SW2 57.6 mm to (108.0, 46.5), turned to -90 degrees
- moved C2 57.5 mm to (112.0, 40.2), turned to -90 degrees
- moved C1 56.7 mm to (109.8, 40.2), turned to -90 degrees
- moved R1 56.2 mm to (107.8, 40.1), turned to 90 degrees
- moved SW1 47.2 mm to (136.7, 46.5), turned to 90 degrees
- moved R6 46.6 mm to (112.2, 50.2), turned to -90 degrees
- moved C3 41.1 mm to (112.2, 44.5), turned to -90 degrees
- moved U2 35.2 mm to (123.2, 46.2)
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Routing:
- net +3V3: track 0.00 -> 84.1 mm, vias 2 -> 0
- net USBD-: track 0.00 -> 37.7 mm
- net USBD+: track 0.00 -> 37.7 mm
- net SDA: track 0.00 -> 20.1 mm
- net SCL: track 0.00 -> 20.0 mm
- net CHIP_PU: track 0.00 -> 16.5 mm
- net Earth: track 0.00 -> 13.3 mm, vias 20 -> 49
- net VCC: track 0.00 -> 13.2 mm, vias 0 -> 3
- net GPIO9: track 0.00 -> 13.1 mm
- net /VBUS: track 0.00 -> 12.6 mm, vias 0 -> 2
- net Net-(J2-CC2): track 0.00 -> 9.46 mm
- net /USBCD-: track 0.00 -> 9.13 mm
- net /USBCD+: track 0.00 -> 8.16 mm
- net Net-(J2-CC1): track 0.00 -> 7.43 mm
- net Net-(U3-ISET): track 0.00 -> 3.46 mm
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- added copper zone on F.Cu, net +3V3
- added copper zone on F.Cu, net /BAT+
- added copper zone on F.Cu, net /VBUS
- added copper zone on F.Cu, net /VBUSF
- added copper zone on F.Cu, net /VIN
- added copper zone on B.Cu, net Earth
- added copper zone on F.Cu, net Earth
- added copper zone on F.Cu, net Net-(U5-L1)
- added copper zone on F.Cu, net Net-(U5-L2)
- added copper zone on F.Cu, net VCC
Other:
- board outline added: 75 x 31.5 mm
- board text added: "+"
- board text added: "-"
- board text added: "3V3"
- board text added: "BOOT"
- board text added: "RESET"

Commit message: Udpated to V3.1
Parts:
- J1: footprint Connector_JST:JST_XH_B2B-XH-A_1x02_P2.50mm_Vertical -> Connector_JST:JST_PH_B2B-PH-K_1x02_P2.00mm_Vertical
- moved J1 0.49 mm to (69.0, 40.7)
Changed lines of the file:
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@@
 		)
 	)
-	(footprint "Connector_JST:JST_XH_B2B-XH-A_1x02_P2.50mm_Vertical"
+	(footprint "Connector_JST:JST_PH_B2B-PH-K_1x02_P2.00mm_Vertical"
 		(layer "F.Cu")
-		(at 69.25 40.25 -90)
-		(descr "JST XH series connector, B2B-XH-A (http://www.jst-mfg.com/product/pdf/eng/eXH.pdf)")
-		(tags "connector JST XH vertical")
+		(at 69.05 40.698438 -90)
+		(descr "JST PH series connector, B2B-PH-K (http://www.jst-mfg.com/product/pdf/eng/ePH.pdf)")
+		(tags "connector JST PH vertical")
 		(property "Reference" "J1"
-			(at 1.25 -3.55 90)
+			(at 1 -2.9 90)
 			(layer "F.SilkS")
 			(hide yes)
@@
 		)
 		(property "Value" "Conn_01x02"
-			(at 1.25 4.6 90)
+			(at 1 4 90)
 			(layer "F.Fab")
 			(effects
@@
 			)
 		)
-		(property "LCSC" "C158012"
-			(at 0 0 270)
-			(unlocked yes)
-			(layer "F.Fab")
-			(hide yes)
-			(effects
-				(font
-					(size 1 1)
-					(thickness 0.15)
-				)
-			)
-		)
-		(property "LCSC Part" ""
+		(property "LCSC Part" "C131337"
 			(at 0 0 270)
 			(unlocked yes)
@@
 		(duplicate_pad_numbers_are_jumpers no)
 		(fp_line
-			(start -1.8 2.75)
-			(end 1.25 2.75)
+			(start -1.45 2.3)
+			(end 3.45 2.3)
 			(stroke
 				(width 0.12)
@@
 		)
 		(fp_line
-			(start 4.3 2.75)
-			(end 1.25 2.75)
+			(start 0.9 2.3)
+			(end 0.9 1.8)
 			(stroke
 				(width 0.12)
@@
 		)
 		(fp_line
-			(start -2.55 -0.2)
-			(end -1.8 -0.2)
+			(start 1 2.3)
+			(end 1 1.8)
 			(stroke
 				(width 0.12)
@@
 		)
 		(fp_line
-			(start -1.8 -0.2)
-			(end -1.8 2.75)
+			(start 3.45 2.3)
+			(end 3.45 -1.2)
 			(stroke
 				(width 0.12)
@@
 		)
 		(fp_line
-			(start 4.3 -0.2)
-			(end 4.3 2.75)
+			(start 0.9 1.8)
+			(end 1.1 1.8)
 			(stroke
 				(width 0.12)
@@
 		)
 		(fp_line
-			(start 5.05 -0.2)
-			(end 4.3 -0.2)
+			(start 1.1 1.8)
+			(end 1.1 2.3)
 			(stroke
 				(width 0.12)
@@
 		)
 		(fp_line
-			(start -2.85 -2.75)
-			(end -2.85 -1.5)
+			(start -2.06 0.8)
+			(end -1.45 0.8)
 			(stroke
 				(width 0.12)
@@
 		)
 		(fp_line
-			(start -1.6 -2.75)
-			(end -2.85 -2.75)
+			(start 4.06 0.8)
+			(end 3.45 0.8)
 			(stroke
 				(width 0.12)
@@
 			(layer "F.SilkS")
 		)
-		(fp_rect
-			(start -2.55 -2.45)
-			(end -0.75 -1.7)
+		(fp_line
+			(start -2.06 -0.5)
+			(end -1.45 -0.5)
 			(stroke
 				(width 0.12)
 				(type solid)
 			)
-			(fill no)
 			(layer "F.SilkS")
 		)
-		(fp_rect
-			(start 0.75 -2.45)
-			(end 1.75 -1.7)
+		(fp_line
+			(start 4.06 -0.5)
+			(end 3.45 -0.5)
 			(stroke
 				(width 0.12)
 				(type solid)
 			)
-			(fill no)
 			(layer "F.SilkS")
 		)
-		(fp_rect
-			(start 3.25 -2.45)
-			(end 5.05 -1.7)
+		(fp_line
+			(start -1.45 -1.2)
+			(end -1.45 2.3)
+			(stroke
+				(width 0.12)
+				(type solid)
+			)
+			(layer "F.SilkS")
+		)
+		(fp_line
+			(start 0.5 -1.2)
+			(end -1.45 -1.2)
+			(stroke
+				(width 0.12)
+				(type solid)
+			)
+			(layer "F.SilkS")
+		)
+		(fp_line
+			(start 1.5 -1.2)
+			(end 1.5 -1.81)
+			(stroke
+				(width 0.12)
+				(type solid)
+			)
+			(layer "F.SilkS")
+		)
+		(fp_line
+			(start 3.45 -1.2)
+			(end 1.5 -1.2)
+			(stroke
+				(width 0.12)
+				(type solid)
+			)
+			(layer "F.SilkS")
+		)
+		(fp_line
+			(start -0.3 -1.81)
+			(end -0.3 -2.01)
+			(stroke
+				(width 0.12)
+				(type solid)
+			)
+			(layer "F.SilkS")
+		)
+		(fp_line
+			(start 0.5 -1.81)
+			(end 0.5 -1.2)
+			(stroke
+				(width 0.12)
+				(type solid)
+			)
+			(layer "F.SilkS")
+		)
+		(fp_line
+			(start -0.3 -1.91)
+			(end -0.6 -1.91)
+			(stroke
+				(width 0.12)
+				(type solid)
+			)
+			(layer "F.SilkS")
+		)
+		(fp_line
+			(start -0.6 -2.01)
+			(end -0.6 -1.81)
+			(stroke
+				(width 0.12)
+				(type solid)
+			)
+			(layer "F.SilkS")
+		)
+		(fp_line
+			(start -0.3 -2.01)
+			(end -0.6 -2.01)
+			(stroke
+				(width 0.12)
+				(type solid)
+			)
+			(layer "F.SilkS")
+		)
+		(fp_line
+			(start -2.36 -2.11)
+			(end -2.36 -0.86)
+			(stroke
+				(width 0.12)
+				(type solid)
+			)
+			(layer "F.SilkS")
+		)
+		(fp_line
+			(start -1.11 -2.11)
+			(end -2.36 -2.11)
 			(stroke
 				(width 0.12)
 				(type solid)
 			)
-			(fill no)
 			(layer "F.SilkS")
 		)
 		(fp_rect
-			(start -2.56 -2.46)
-			(end 5.06 3.51)
+			(start -2.06 -1.81)
+			(end 4.06 2.91)
 			(stroke
 				(width 0.12)
@@
 		)
 		(fp_rect
-			(start -2.95 -2.85)
-			(end 5.45 3.9)
+			(start -2.45 -2.2)
+			(end 4.45 3.3)
 			(stroke
 				(width 0.05)
@@
 		)
 		(fp_line
-			(start 0 -1.35)
-			(end 0.625 -2.35)
+			(start -2.36 -2.11)
+			(end -2.36 -0.86)
 			(stroke
 				(width 0.1)
@@
 		)
 		(fp_line
-			(start -0.625 -2.35)
-			(end 0 -1.35)
+			(start -1.11 -2.11)
+			(end -2.36 -2.11)
 			(stroke
 				(width 0.1)
@@
 		)
 		(fp_rect
-			(start -2.45 -2.35)
-			(end 4.95 3.4)
+			(start -1.95 -1.7)
+			(end 3.95 2.8)
 			(stroke
 				(width 0.1)
@@
 		)
 		(fp_text user "${REFERENCE}"
-			(at 1.25 2.7 90)
+			(at 1 1.5 90)
 			(layer "F.Fab")
 			(effects
@@
 		(pad "1" thru_hole roundrect
 			(at 0 0 270)
-			(size 1.7 2)
-			(drill 1)
+			(size 1.2 1.75)
+			(drill 0.75)
 			(layers "*.Cu" "*.Mask")
 			(remove_unused_layers no)
-			(roundrect_rratio 0.147059)
+			(roundrect_rratio 0.208333)
 			(net "Earth")
 			(pinfunction "Pin_1_1")
 			(pintype "passive")
-			(zone_connect 2)
 		)
 		(pad "2" thru_hole oval
-			(at 2.5 0 270)
-			(size 1.7 2)
-			(drill 1)
+			(at 2 0 270)
+			(size 1.2 1.75)
+			(drill 0.75)
 			(layers "*.Cu" "*.Mask")
 			(remove_unused_layers no)
@@
 			(pinfunction "Pin_2_2")
 			(pintype "passive")
-			(zone_connect 2)
 		)
 		(embedded_fonts no)
-		(model "${KICAD10_3DMODEL_DIR}/Connector_JST.3dshapes/JST_XH_B2B-XH-A_1x02_P2.50mm_Vertical.step"
+		(model "${KICAD10_3DMODEL_DIR}/Connector_JST.3dshapes/JST_PH_B2B-PH-K_1x02_P2.00mm_Vertical.step"
 			(offset
 				(xyz 0 0 0)
@@
 		(layer "Edge.Cuts")
 	)
-	(gr_text "-"
-		(at 72.75 37.75 0)
+	(gr_text "+"
+		(at 71.9 44.2 0)
 		(layer "F.SilkS")
 		(effects
@@
 		)
 	)
-	(gr_text "+"
-		(at 72.75 44.75 0)
+	(gr_text "-"
+		(at 72 38.9 0)
 		(layer "F.SilkS")
 		(effects
@@
 	)
 	(via
-		(at 69.225 38.5)
+		(at 69.025 38.948438)
 		(size 0.6)
 		(drill 0.3)
@@
 	)
 	(via
-		(at 67.475 40.25)
+		(at 67.275 40.698438)
 		(size 0.6)
 		(drill 0.3)
@@
 	)
 	(via
-		(at 70.975 40.25)
+		(at 70.775 40.698438)
 		(size 0.6)
 		(drill 0.3)
@@
 		(polygon
 			(pts
-				(xy 76.8 45.1) (xy 76.792828 41.880855) (xy 68.211907 41.867478) (xy 68.209148 43.637337) (xy 75.3 43.6)
+				(xy 76.8 45.1) (xy 76.79244 41.706692) (xy 67.962198 41.69306) (xy 67.959166 43.638519) (xy 75.3 43.6)
 				(xy 76 44.3) (xy 76 45.1)
 			)
