File: temp-humidity sensor.kicad_sch (KiCad schematic)
At the start: 31 parts, among them J1 USB_C_Receptacle_USB2.0_16P, J2 Conn_01x02, SW1 SW_Push, SW2 SW_Push, U1 SHT4x, U2 ESP32-C6-WROOM-1, U3 USBLC6-2SC6, U4 BQ24074RGT

Commit message: Finished Schematic
Parts:
- removed R1: 0R, Resistor_SMD:R_0603_1608Metric, symbol Device:R
- removed R3: 10K, Resistor_SMD:R_0603_1608Metric, symbol Device:R
- added C10, C7, C9: 10u, Capacitor_SMD:C_0603_1608Metric, symbol Device:C
- added C8: 100n, Capacitor_SMD:C_0603_1608Metric, symbol Device:C
- added L1: 1.5u, Inductor_SMD:L_Changjiang_FXL0630, symbol Device:L
- added R6: 10K, Resistor_SMD:R_0603_1608Metric, symbol Device:R
- added SW3: SS-12D01-G040, LCSC:SW-TH_SS-12D01-GX, symbol LCSC:SS-12D01-G040
- added U5: TPS63031DSK, Package_SON:WSON-10-1EP_2.5x2.5mm_P0.5mm_EP1.2x2mm, symbol Regulator_Switching:TPS63031DSK
- C1: LCSC (none) -> C19702
- C2, C4: LCSC (none) -> C77055
- C3: LCSC (none) -> C59302
- C5: renamed from C6; LCSC (none) -> C59302
- C6: renamed from C5; LCSC (none) -> C19702
- D1: footprint (none) -> LED_SMD:LED_0805_2012Metric; LCSC (none) -> C19171391
- J1: renamed from J2; LCSC (none) -> C158012
- J2: renamed from J1; footprint (none) -> Connector_USB:USB_C_Receptacle_G-Switch_GT-USB-7010ASV
- R1: renamed from R2; LCSC (none) -> C2930027
- R12: LCSC (none) -> C2930027
- R13: renamed from R10; LCSC (none) -> C2907129
- R14: renamed from R11; LCSC (none) -> C2907129
- R2: renamed from R7; LCSC (none) -> C2930027
- R3: renamed from R6; LCSC (none) -> C2930027
- R4, R5: LCSC (none) -> C2907129
- R7: renamed from R8; LCSC (none) -> C2907044
- R8: renamed from R13; LCSC (none) -> C2930027
- R9: LCSC (none) -> C2907044
- U1: LCSC (none) -> C54946589
- U3: renamed from U4; LCSC (none) -> C54313
- renumbered R14 to R10, R15 to R11, U3 to U4
Connections:
- net BT+ is gone; now on net BAT+: BT1.1 (+), J1.2 (Pin_2)
- net ESP3V3 is gone; now on net +3V3: C2.1, R1.2, U2.2 (3V3)
- net +3V3: now also R6.2, SW3.3
- net Earth: now also C10.2, C7.2, C8.2, C9.2, U5.11 (PGND), U5.3 (PGND), U5.9 (GND)
- net GPIO8: now also R6.1
- net VOUT: now also C10.1, C9.1, SW3.2, U5.1 (VOUT), U5.10 (FB); no longer R12.2, U3.10 (OUT), U3.11 (OUT), U3.5 (EN2)
- net SCLF: now reaches R3.1, R4.1, U1.2 (SCL)
- net SDAF: now reaches R2.1, R5.1, U1.1 (SDA)
- net BT- renamed BAT-
- net GPIO12 renamed USBD-
- net GPIO13 renamed USBD+
- net GPIO6 renamed SDA
- net GPIO7 renamed SCL
- new net: L1.1, U5.4 (L1)
- new net: L1.2, U5.2 (L2)
- new net: C8.1, U5.6 (EN), U5.7 (PS/SYNC), U5.8 (VINA)
- new net +5V: C7.1, R12.2, U3.10 (OUT), U3.11 (OUT), U3.5 (EN2), U5.5 (VIN)
- no-connect marks 21 -> 23
Other:
- note added: "BUCK BOOST"
- moved on the sheet: BT1, C4, C5, C6, D1, J1, J2, R10, R11, R12, R13, R14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

Commit message: Working On PCB
Parts:
- added C11, C12: 470n, Capacitor_SMD:C_0603_1608Metric, symbol Device:C
- added R15: 0R, Resistor_SMD:R_0603_1608Metric, symbol Device:R
- C10: value 10u -> 100n
Connections:
- net BAT- is gone; now on net Earth: BT1.2 (-), J1.1 (Pin_1)
- net Earth: now also C11.2, C12.2
- net GPIO9: now also U2.15 (GPIO9)
- net VBUS: now also C11.1, R15.2; no longer C5.1, U3.13 (IN)
- new net VBUSF: C12.1, C5.1, R15.1, U3.13 (IN)
- no-connect marks 23 -> 22

Commit message: Finished Design
Parts:
- removed R13, R14: 22R, Resistor_SMD:R_0603_1608Metric, symbol Device:R
- added TP2, TP3, TP4, TP5, TP6: TestPoint, TestPoint:TestPoint_Pad_D1.0mm, symbol Connector:TestPoint
- SW3: footprint LCSC:SW-TH_SS-12D01-GX -> easyeda2kicad:SW-TH_SS-12D01-GX
Connections:
- net +3V3: now also TP2.1, TP6.1
- net BAT+: now also TP5.1
- net USBD+: now also U4.4 (I/O2)
- net USBD-: now also U4.6 (I/O1)
- net VOUT: now also TP4.1
- net +5V renamed VSYS
- net VSYS: now also TP3.1

Commit message: V3
Parts:
- removed SW3: SS-12D01-G040, easyeda2kicad:SW-TH_SS-12D01-GX, symbol LCSC:SS-12D01-G040
- removed TP6: TestPoint, TestPoint:TestPoint_Pad_D1.0mm, symbol Connector:TestPoint
- added U6: SS12D10G5, easyeda2kicad:SW-TH_SHOU-HAN_SS12D10G4, symbol easyeda2kicad:SS12D10G5
- C1, C7, C9: footprint Capacitor_SMD:C_0603_1608Metric -> Capacitor_SMD:C_0805_2012Metric; LCSC C19702 -> C5448891
- C10: value 100n -> 10u; footprint Capacitor_SMD:C_0603_1608Metric -> Capacitor_SMD:C_0805_2012Metric; LCSC C19702 -> C5448891
- C2: footprint Capacitor_SMD:C_0603_1608Metric -> Capacitor_SMD:C_0805_2012Metric; LCSC C77055 -> C111492
- C3: LCSC C59302 -> C106248
- C5: footprint Capacitor_SMD:C_0603_1608Metric -> Capacitor_SMD:C_0805_2012Metric; LCSC C59302 -> C91185
- C6: value 10u -> 4.7u; footprint Capacitor_SMD:C_0603_1608Metric -> Capacitor_SMD:C_0805_2012Metric; LCSC C19702 -> C354262
- R10: value 1.2K -> 1.3K; LCSC C2906976 -> C2906977
- R11: value 680R -> 698R; LCSC C23228 -> C7467401
- U2: footprint PCM_Espressif_1:ESP32-C6-WROOM-1 -> PCM_Espressif:ESP32-C6-WROOM-1
Connections:
- net VOUT is gone; now on net +3V3: C10.1, C9.1, TP4.1, U5.1 (VOUT), U5.10 (FB)
- net VSYS renamed VCC
- net VCC: now also U6.2; no longer C7.1, U5.5 (VIN)
- new net VIN: C7.1, U5.5 (VIN), U6.3
Other:
- note added: "Around 1.2A"
- note removed: "Around 1.3A"
- moved on the sheet: BT1, C1, C11, C12, C2, C3, C4, C5, C6, C7, C8, D1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

Commit message: Update to V3
Parts:
- added TP6, TP7, TP8, TP9: TestPoint, TestPoint:TestPoint_Pad_D1.0mm, symbol Connector:TestPoint
Connections:
- net Earth: now also TP6.1, TP7.1, TP8.1, TP9.1
Other:
- moved on the sheet: BT1, J1, SW1, SW2

Commit message: Udpated to V3.1
Parts:
- J1: footprint Connector_JST:JST_XH_B2B-XH-A_1x02_P2.50mm_Vertical -> Connector_JST:JST_PH_B2B-PH-K_1x02_P2.00mm_Vertical; LCSC C158012 -> (none); LCSC Part (none) -> C131337
- TP2, TP3, TP4, TP5, TP6, TP7, TP8, TP9: now left out of the parts list
Changed lines of the file:
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@@
 		(body_style 1)
 		(exclude_from_sim no)
-		(in_bom yes)
+		(in_bom no)
 		(on_board yes)
 		(in_pos_files yes)
@@
 		(body_style 1)
 		(exclude_from_sim no)
-		(in_bom yes)
+		(in_bom no)
 		(on_board yes)
 		(in_pos_files yes)
@@
 		(body_style 1)
 		(exclude_from_sim no)
-		(in_bom yes)
+		(in_bom no)
 		(on_board yes)
 		(in_pos_files yes)
@@
 		(body_style 1)
 		(exclude_from_sim no)
-		(in_bom yes)
+		(in_bom no)
 		(on_board yes)
 		(in_pos_files yes)
@@
 		(body_style 1)
 		(exclude_from_sim no)
-		(in_bom yes)
+		(in_bom no)
 		(on_board yes)
 		(in_pos_files yes)
@@
 		(body_style 1)
 		(exclude_from_sim no)
-		(in_bom yes)
+		(in_bom no)
 		(on_board yes)
 		(in_pos_files yes)
@@
 		(body_style 1)
 		(exclude_from_sim no)
-		(in_bom yes)
+		(in_bom no)
 		(on_board yes)
 		(in_pos_files yes)
@@
 			)
 		)
-		(property "Footprint" "Connector_JST:JST_XH_B2B-XH-A_1x02_P2.50mm_Vertical"
+		(property "Footprint" "Connector_JST:JST_PH_B2B-PH-K_1x02_P2.00mm_Vertical"
 			(at 20.32 187.96 0)
 			(hide yes)
@@
 			)
 		)
-		(property "Datasheet" "https://www.lcsc.com/product-detail/C158012.html?s_z=n_q_C158012&globalKeyword=C158012"
+		(property "Datasheet" "https://www.lcsc.com/product-detail/C131337.html?s_z=n_q_C131337&globalKeyword=C131337"
 			(at 20.32 187.96 0)
 			(hide yes)
@@
 			)
 		)
-		(property "LCSC" "C158012"
-			(at 20.32 187.96 0)
-			(hide yes)
-			(show_name no)
-			(do_not_autoplace no)
-			(effects
-				(font
-					(size 1.27 1.27)
-				)
-			)
-		)
-		(property "LCSC Part" ""
+		(property "LCSC Part" "C131337"
 			(at 20.32 187.96 0)
 			(hide yes)
@@
 		(body_style 1)
 		(exclude_from_sim no)
-		(in_bom yes)
+		(in_bom no)
 		(on_board yes)
 		(in_pos_files yes)
