File: temp-humidity sensor.kicad_sch (KiCad schematic)
At the start: 46 parts, among them J1 Conn_01x02, J2 USB_C_Receptacle_USB2.0_16P, SW1 SW_Push, SW2 SW_Push, U1 SHT4x, U2 ESP32-C6-WROOM-1, U3 BQ24074RGT, U4 USBLC6-2SC6, U5 TPS63031DSK, U6 SS12D10G5

Commit message: Improved design
Parts:
- removed TP4: TestPoint, TestPoint:TestPoint_Pad_D1.0mm, symbol Connector:TestPoint
- removed U6: SS12D10G5, easyeda2kicad:SW-TH_SHOU-HAN_SS12D10G4, symbol easyeda2kicad:SS12D10G5
- added C13: 4.7u, Capacitor_SMD:C_0805_2012Metric, symbol Device:C
- added H1, H2, H3, H4: MountingHole, MountingHole:MountingHole_3.2mm_M3_ISO7380_Pad_TopBottom, symbol Mechanical:MountingHole_Pad
- added SW3: SW_SPDT, Button_Switch_THT:SW_Slide_SPDT_Straight_CK_OS102011MS2Q, symbol Switch:SW_SPDT
- SW1, SW2: footprint Button_Switch_SMD:SW_SPST_PTS647_Sx38 -> Button_Switch_SMD:SW_Push_SPST_NO_Alps_SKRK
- renumbered R9 to R11, R7 to R12, R12 to R7, R11 to R9
Connections:
- net VIN is gone; now on net VCC: C7.1, U5.5 (VIN)
- net BAT+: now also J1.1 (Pin_1); no longer J1.2 (Pin_2)
- net Earth: now also J1.2 (Pin_2), C13.2, H1.1, H2.1, H3.1, H4.1, SW3.3 (C); no longer J1.1 (Pin_1)
- net VCC: now also C13.1
- net VINA: now reaches C8.1, U5.7 (PS/SYNC), U5.8 (VINA)
- net VINA: now also SW3.2 (B); no longer U5.6 (EN)
- new net PWR_EN: SW3.1 (A), U5.6 (EN)
- no-connect marks 22 -> 21
Other:
- moved on the sheet: C1, C10, C2, C3, C7, C8, C9, J1, R1, R6, U2
